File: PSU.sch (KiCad schematic (older format))
At the start: 0 parts

Commit message: Imported CAN and PSU blocks from infrastructure rep
Parts:
- added C? (x3): 1u, symbol Device:C
- added C? (x2): 100n, symbol Device:C
- added D?: D_Schottky, symbol Device:D_Schottky
- added D? (x2): D_TVS, symbol Device:D_TVS
- added D?: RED, symbol Device:LED
- added F?: Fuse, symbol Device:Fuse
- added FB?: Ferrite_Bead, symbol Device:Ferrite_Bead
- added R?: 510, symbol Device:R
- added U?: ADP150AUJZ-3.3-R7, Package_TO_SOT_SMD:SOT-23-5, symbol KTHFS:ADP150AUJZ-3.3-R7
- added VR?: Wurth-FDSM, KTHFS:Wurth-FDSM, symbol KTHFS:Wurth-FDSM
Connections:
- new net: FB?.2, VR?.3 (OUT)
- new net: D?.1 (K), F?.2
- new net: D?.1 (K), R?.1
- new net +24V: C?.1, D?.1 (A1), F?.1, VR?.1 (IN)
- new net +3V3: C?.1, C?.1, U?.5 (VOUT)
- new net +5V: C?.1, C?.1, D?.1 (A1), D?.2 (A), FB?.1, U?.1 (VIN), U?.3 (EN)
- new net GND: C?.2, C?.2, C?.2, C?.2, C?.2, D?.2 (A2), D?.2 (A2), R?.2, U?.2 (GND), VR?.2 (GND)
- new net battery_in: D?.2 (A)
Other:
- note added: "tells ERC that this is\na power source"
