File: PA.sch (KiCad schematic (older format))
At the start: 31 parts, among them J6 RF_Shield_One_Piece, U4 CC1190RGVR

Commit message: Small changes to schematic
Other:
- note added: "SAW filter is used to pass regulation by\ndecreasing phasenoise at the band edges.\nIf not used output power may have to be reduced."
- note added: "Shield for PA might not be neccecairy"
- note removed: "Reference design by TI:\nhttps://www.ti.com/lit/df/tidr235/tidr235.pdf?ts=1612292840663&ref_url=https%253A%252F%252Fwww.google.com%252F"
- note removed: "SAW filter is used to pass regulation by\ndecreasing phasenoise at the band edges.\nIf not used output power has to be reduced."
- moved on the sheet: J6, R14, R15, R16
Changed lines of the file:
@@
 Comment4 ""
 $EndDescr
-Text Notes 550  750  0    59   ~ 0
-Reference design by TI:\nhttps://www.ti.com/lit/df/tidr235/tidr235.pdf?ts=1612292840663&ref_url=https%253A%252F%252Fwww.google.com%252F
-$Comp
-L Device:RF_Shield_One_Piece J6
-U 1 1 602F38D4
-P 2100 6600
-F 0 "J6" H 2050 7150 50  0000 L CNN
-F 1 "RF_Shield_One_Piece" H 1700 7050 50  0000 L CNN
-F 2 "" H 2100 6500 50  0001 C CNN
-F 3 "~" H 2100 6500 50  0001 C CNN
-	1    2100 6600
-	1    0    0    -1
-$EndComp
 $Comp
 L power:GND #PWR059
 U 1 1 602F428E
-P 2100 7000
-F 0 "#PWR059" H 2100 6750 50  0001 C CNN
-F 1 "GND" H 2105 6827 50  0000 C CNN
-F 2 "" H 2100 7000 50  0001 C CNN
-F 3 "" H 2100 7000 50  0001 C CNN
-	1    2100 7000
-	1    0    0    -1
-$EndComp
-Text Notes 8450 2850 0    39   ~ 0
+P 3750 6950
+F 0 "#PWR059" H 3750 6700 50  0001 C CNN
+F 1 "GND" H 3755 6777 50  0000 C CNN
+F 2 "" H 3750 6950 50  0001 C CNN
+F 3 "" H 3750 6950 50  0001 C CNN
+	1    3750 6950
+	1    0    0    -1
+$EndComp
+Text Notes 8450 2875 0    59   ~ 0
 SAW filter may not be neccecairy. \nExact component not decided yet.
 $Comp
@@
 	1    0    0    -1
 $EndComp
-Text Notes 9300 4000 0    39   ~ 0
-SAW filter is used to pass regulation by\ndecreasing phasenoise at the band edges.\nIf not used output power has to be reduced.
+Text Notes 8425 4625 0    59   ~ 0
+SAW filter is used to pass regulation by\ndecreasing phasenoise at the band edges.\nIf not used output power may have to be reduced.
 Connection ~ 9450 3600
 Wire Wire Line
@@
 $EndComp
 Wire Wire Line
-	5350 3850 6200 3850
-Wire Wire Line
 	5350 3050 5350 3250
 Wire Wire Line
@@
 	1    0    0    -1
 $EndComp
-Wire Wire Line
-	6200 3150 6150 3150
-Text HLabel 5500 1600 0    59   Input ~ 0
+Text HLabel 5450 1600 0    59   Input ~ 0
 PA_EN
-Text HLabel 5500 1500 0    59   Input ~ 0
+Text HLabel 5450 1500 0    59   Input ~ 0
 LNA_EN
-Text HLabel 5500 1400 0    59   Input ~ 0
+Text HLabel 5450 1400 0    59   Input ~ 0
 HGM
-Wire Wire Line
-	5850 3450 5850 4200
 Wire Wire Line
 	5200 3650 6200 3650
@@
 L Device:R R14
 U 1 1 601E98C3
-P 5650 2350
-F 0 "R14" H 5720 2396 50  0000 L CNN
-F 1 "10k" H 5720 2305 50  0000 L CNN
-F 2 "" V 5580 2350 50  0001 C CNN
-F 3 "~" H 5650 2350 50  0001 C CNN
-	1    5650 2350
+P 5600 2350
+F 0 "R14" H 5670 2396 50  0000 L CNN
+F 1 "10k" H 5670 2305 50  0000 L CNN
+F 2 "" V 5530 2350 50  0001 C CNN
+F 3 "~" H 5600 2350 50  0001 C CNN
+	1    5600 2350
 	1    0    0    -1
 $EndComp
@@
 L Device:R R15
 U 1 1 601EB9A5
-P 5900 2350
-F 0 "R15" H 5970 2396 50  0000 L CNN
-F 1 "10k" H 5970 2305 50  0000 L CNN
-F 2 "" V 5830 2350 50  0001 C CNN
-F 3 "~" H 5900 2350 50  0001 C CNN
-	1    5900 2350
+P 5850 2350
+F 0 "R15" H 5920 2396 50  0000 L CNN
+F 1 "10k" H 5920 2305 50  0000 L CNN
+F 2 "" V 5780 2350 50  0001 C CNN
+F 3 "~" H 5850 2350 50  0001 C CNN
+	1    5850 2350
 	1    0    0    -1
 $EndComp
@@
 L Device:R R16
 U 1 1 601EFB2B
-P 6150 2350
-F 0 "R16" H 6220 2396 50  0000 L CNN
-F 1 "10k" H 6220 2305 50  0000 L CNN
-F 2 "" V 6080 2350 50  0001 C CNN
-F 3 "~" H 6150 2350 50  0001 C CNN
-	1    6150 2350
-	1    0    0    -1
-$EndComp
-Wire Wire Line
-	5500 1400 5650 1400
-Wire Wire Line
-	5650 1400 5650 2200
-Wire Wire Line
-	5500 1500 5900 1500
-Wire Wire Line
-	5900 1500 5900 2200
-Wire Wire Line
-	5500 1600 6150 1600
-Wire Wire Line
-	6150 1600 6150 2200
-Wire Wire Line
-	5650 2500 5650 2850
-Wire Wire Line
-	5650 2850 6200 2850
-Wire Wire Line
-	5900 2950 6200 2950
-Wire Wire Line
-	5900 2500 5900 2950
-Wire Wire Line
-	6150 2500 6150 3150
+P 6100 2350
+F 0 "R16" H 6170 2396 50  0000 L CNN
+F 1 "10k" H 6170 2305 50  0000 L CNN
+F 2 "" V 6030 2350 50  0001 C CNN
+F 3 "~" H 6100 2350 50  0001 C CNN
+	1    6100 2350
+	1    0    0    -1
+$EndComp
+Wire Wire Line
+	5450 1400 5600 1400
+Wire Wire Line
+	5600 1400 5600 2200
+Wire Wire Line
+	5450 1500 5850 1500
+Wire Wire Line
+	5850 1500 5850 2200
+Wire Wire Line
+	5450 1600 6100 1600
+Wire Wire Line
+	6100 1600 6100 2200
+Wire Wire Line
+	5600 2500 5600 2850
+Wire Wire Line
+	5850 2500 5850 2950
+Wire Wire Line
+	6100 2500 6100 3150
 $Comp
 L Device:C C16
@@
 Wire Wire Line
 	3650 3050 4100 3050
+Wire Wire Line
+	5600 2850 6200 2850
+Wire Wire Line
+	5850 2950 6200 2950
+Wire Wire Line
+	6100 3150 6200 3150
+Wire Wire Line
+	5850 3450 5850 4200
+Wire Wire Line
+	5350 3850 6200 3850
+$Comp
+L Device:RF_Shield_One_Piece J6
+U 1 1 602F38D4
+P 3750 6550
+F 0 "J6" H 3700 7100 50  0000 L CNN
+F 1 "RF_Shield_One_Piece" H 3350 7000 50  0000 L CNN
+F 2 "" H 3750 6450 50  0001 C CNN
+F 3 "~" H 3750 6450 50  0001 C CNN
+	1    3750 6550
+	1    0    0    -1
+$EndComp
+Text Notes 2925 5850 0    59   ~ 0
+Shield for PA might not be neccecairy
 $EndSCHEMATC

Commit message: Changes to PA layout
Parts:
- removed C12: 47p, symbol Device:C
- removed C14, C16: 12p, symbol Device:C
- removed C15: 2.7p, symbol Device:C
- removed C70: 15p, symbol Device:C
- removed J6: RF_Shield_One_Piece, symbol Device:RF_Shield_One_Piece
- removed L4: 7.5n, symbol Device:L
- removed L5: 2.7n, symbol Device:L
- removed L6: 22n, symbol Device:L
- removed L7: 10n, symbol Device:L
- removed L8: 1.5n, symbol Device:L
- removed L9: 15n, symbol Device:L
- removed R14, R15, R16: 10k, symbol Device:R
- removed R4: 3.3k, symbol Device:R
- removed R5: 47, symbol Device:R
- removed U4: CC1190RGVR, QFN65P400X400X100-17N, symbol CC1190RGVR:CC1190RGVR
- added C? (x2): 47p, symbol Device:C
- added C? (x2): 12p, symbol Device:C
- added C?: 2.7p, symbol Device:C
- added C?: 15p, symbol Device:C
- added C?: 27p, symbol Device:C
- added C?: 1u, symbol Device:C
- added C?: 1n, symbol Device:C
- added IC?: CC1190, QFN65P400X400X100-17N, symbol KTHFS:CC1190
- added L?: 7.5n, symbol Device:L
- added L?: 2.7n, symbol Device:L
- added L?: L, symbol Device:L
- added L?: 15n, symbol Device:L
- added L?: 22n, symbol Device:L
- added L?: 10n, symbol Device:L
- added R? (x3): 10k, symbol Device:R
- added R?: 47, symbol Device:R
- added R?: 3.3k, symbol Device:R
- C10, C11, C13, C17, C7, C8, C9: footprint (none) -> Capacitor_SMD:C_0603_1608Metric
- L1, L2, L3: footprint (none) -> Inductor_SMD:L_0603_1608Metric
- R7: footprint (none) -> Resistor_SMD:R_0603_1608Metric
Connections:
- net GND: now also C?.2, C?.2, C?.2, C?.2, C?.2, C?.2, IC?.1 (GND@1), IC?.12 (GND@4), IC?.17 (GND-PL), IC?.3 (GND@2), IC?.9 (GND@3), R?.2
- net HGM: now also IC?.6 (HGM), R?.1, R?.2
- net LNA_EN: now also IC?.7 (LNA-EN), R?.1, R?.2
- net PA_EN: now also IC?.8 (PA-EN), R?.1, R?.2
- net at C13.1, L3.2, TP1.1: now also C?.1, C?.1, C?.1, C?.1, L?.1, L?.1, L?.2, R?.1
- net at C10.1, C9.1, L2.2: now also C?.2, L?.1
- net at C17.1, FL1.1, R7.2: now also L?.1
- new net: IC?.10 (LNA-OUT), IC?.11 (PA-IN), L?.2
- new net: C?.1, IC?.13 (VDD-LNA), L?.1
- new net: IC?.14 (BIAS), R?.1
- new net: IC?.15 (VDD-PA2), R?.2
- new net: IC?.16 (VDD-PA1), L?.2
- new net: C?.1, IC?.2 (PA-OUT), L?.1, L?.2
- new net: C?.2, C?.2, IC?.4 (TR-SW)
- new net: C?.1, IC?.5 (LNA-IN)
- new net: C?.1, L?.2 (x2)
Other:
- note removed: "Shield for PA might not be neccecairy"
- moved on the sheet: C10, C11, C13, C17, C7, C8, C9, FL1, L1, L2, L3, R7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
