File: PA.sch (KiCad schematic (older format))
At the start: 34 parts

Commit message: Changed to F4 MCU
Parts:
- gave numbers to parts that had none: 21
Changed lines of the file:
@@
 LNA_EN
 $Comp
-L Device:R R?
+L Device:R R9
 U 1 1 6051AA9E
 P 5625 7100
-F 0 "R?" H 5555 7054 50  0000 R CNN
+F 0 "R9" H 5555 7054 50  0000 R CNN
 F 1 "10k" H 5555 7145 50  0000 R CNN
 F 2 "" V 5555 7100 50  0001 C CNN
@@
 $EndComp
 $Comp
-L Device:R R?
+L Device:R R11
 U 1 1 6051F9F3
 P 5900 7100
-F 0 "R?" H 5830 7054 50  0000 R CNN
+F 0 "R11" H 5830 7054 50  0000 R CNN
 F 1 "10k" H 5830 7145 50  0000 R CNN
 F 2 "" V 5830 7100 50  0001 C CNN
@@
 $EndComp
 $Comp
-L Device:R R?
+L Device:R R12
 U 1 1 6052394F
 P 6200 7100
-F 0 "R?" H 6130 7054 50  0000 R CNN
+F 0 "R12" H 6130 7054 50  0000 R CNN
 F 1 "10k" H 6130 7145 50  0000 R CNN
 F 2 "" V 6130 7100 50  0001 C CNN
@@
 	4000 1750 3900 1750
 $Comp
-L Device:L L?
+L Device:L L4
 U 1 1 605C08A1
 P 3750 1750
-F 0 "L?" V 3940 1750 50  0000 C CNN
+F 0 "L4" V 3940 1750 50  0000 C CNN
 F 1 "L" V 3849 1750 50  0000 C CNN
 F 2 "" H 3750 1750 50  0001 C CNN
@@
 ANTENNA_OUT
 $Comp
-L KTHFS:CC1190 IC?
+L KTHFS:CC1190 IC1
 U 1 1 603D6DFF
 P 6250 2775
-F 0 "IC?" H 6050 3340 50  0000 C CNN
+F 0 "IC1" H 6050 3340 50  0000 C CNN
 F 1 "CC1190" H 6050 3249 50  0000 C CNN
 F 2 "QFN65P400X400X100-17N" H 5750 3375 50  0001 L BNN
@@
 	6750 3675 6750 3800
 $Comp
-L power:GND #PWR?
+L power:GND #PWR010
 U 1 1 6043B402
 P 6750 3800
-F 0 "#PWR?" H 6750 3550 50  0001 C CNN
+F 0 "#PWR010" H 6750 3550 50  0001 C CNN
 F 1 "GND" H 6755 3627 50  0000 C CNN
 F 2 "" H 6750 3800 50  0001 C CNN
@@
 $EndComp
 $Comp
-L Device:L L?
+L Device:L L7
 U 1 1 604424D7
 P 6225 5300
-F 0 "L?" H 6277 5346 50  0000 L CNN
+F 0 "L7" H 6277 5346 50  0000 L CNN
 F 1 "7.5n" H 6277 5255 50  0000 L CNN
 F 2 "" H 6225 5300 50  0001 C CNN
@@
 $EndComp
 $Comp
-L Device:C C?
+L Device:C C15
 U 1 1 60442C5F
 P 6225 5675
-F 0 "C?" H 6340 5721 50  0000 L CNN
+F 0 "C15" H 6340 5721 50  0000 L CNN
 F 1 "12p" H 6340 5630 50  0000 L CNN
 F 2 "" H 6263 5525 50  0001 C CNN
@@
 Connection ~ 6225 4950
 $Comp
-L Device:C C?
+L Device:C C18
 U 1 1 6045393A
 P 8075 6050
-F 0 "C?" V 7823 6050 50  0000 C CNN
+F 0 "C18" V 7823 6050 50  0000 C CNN
 F 1 "12p" V 7914 6050 50  0000 C CNN
 F 2 "" H 8113 5900 50  0001 C CNN
@@
 	8325 2675 6750 2675
 $Comp
-L Device:C C?
+L Device:C C16
 U 1 1 60441DC2
 P 6850 4950
-F 0 "C?" V 6598 4950 50  0000 C CNN
+F 0 "C16" V 6598 4950 50  0000 C CNN
 F 1 "47p" V 6689 4950 50  0000 C CNN
 F 2 "" H 6888 4800 50  0001 C CNN
@@
 	6225 4950 6700 4950
 $Comp
-L Device:L L?
+L Device:L L9
 U 1 1 60468B05
 P 8550 2675
-F 0 "L?" H 8602 2721 50  0000 L CNN
+F 0 "L9" H 8602 2721 50  0000 L CNN
 F 1 "2.7n" H 8602 2630 50  0000 L CNN
 F 2 "" H 8550 2675 50  0001 C CNN
@@
 $EndComp
 $Comp
-L Device:C C?
+L Device:C C38
 U 1 1 60468FA9
 P 8550 3075
-F 0 "C?" H 8665 3121 50  0000 L CNN
+F 0 "C38" H 8665 3121 50  0000 L CNN
 F 1 "2.7p" H 8665 3030 50  0000 L CNN
 F 2 "" H 8588 2925 50  0001 C CNN
@@
 	8550 2925 8550 2825
 $Comp
-L power:GND #PWR?
+L power:GND #PWR012
 U 1 1 6046D36E
 P 8550 3225
-F 0 "#PWR?" H 8550 2975 50  0001 C CNN
+F 0 "#PWR012" H 8550 2975 50  0001 C CNN
 F 1 "GND" H 8555 3052 50  0000 C CNN
 F 2 "" H 8550 3225 50  0001 C CNN
@@
 	3225 2975 5350 2975
 $Comp
-L Device:C C?
+L Device:C C12
 U 1 1 605C1163
 P 3475 2000
-F 0 "C?" H 3590 2046 50  0000 L CNN
+F 0 "C12" H 3590 2046 50  0000 L CNN
 F 1 "15p" H 3590 1955 50  0000 L CNN
 F 2 "" H 3513 1850 50  0001 C CNN
@@
 $EndComp
 $Comp
-L power:GND #PWR?
+L power:GND #PWR05
 U 1 1 605C6C9D
 P 3475 2150
-F 0 "#PWR?" H 3475 1900 50  0001 C CNN
+F 0 "#PWR05" H 3475 1900 50  0001 C CNN
 F 1 "GND" H 3480 1977 50  0000 C CNN
 F 2 "" H 3475 2150 50  0001 C CNN
@@
 	4250 1850 4250 1750
 $Comp
-L Device:C C?
+L Device:C C14
 U 1 1 60614293
 P 4250 2000
-F 0 "C?" H 4365 2046 50  0000 L CNN
+F 0 "C14" H 4365 2046 50  0000 L CNN
 F 1 "27p" H 4365 1955 50  0000 L CNN
 F 2 "" H 4288 1850 50  0001 C CNN
@@
 $EndComp
 $Comp
-L power:GND #PWR?
+L power:GND #PWR08
 U 1 1 60614299
 P 4250 2150
-F 0 "#PWR?" H 4250 1900 50  0001 C CNN
+F 0 "#PWR08" H 4250 1900 50  0001 C CNN
 F 1 "GND" H 4255 1977 50  0000 C CNN
 F 2 "" H 4250 2150 50  0001 C CNN
@@
 	4250 1750 4750 1750
 $Comp
-L Device:L L?
+L Device:L L6
 U 1 1 6061CE76
 P 5050 2175
-F 0 "L?" H 5102 2221 50  0000 L CNN
+F 0 "L6" H 5102 2221 50  0000 L CNN
 F 1 "15n" H 5102 2130 50  0000 L CNN
 F 2 "" H 5050 2175 50  0001 C CNN
@@
 $EndComp
 $Comp
-L Device:R R?
+L Device:R R4
 U 1 1 6061D4CC
 P 4750 2175
-F 0 "R?" H 4820 2221 50  0000 L CNN
+F 0 "R4" H 4820 2221 50  0000 L CNN
 F 1 "47" H 4820 2130 50  0000 L CNN
 F 2 "" V 4680 2175 50  0001 C CNN
@@
 	4750 2575 4750 2325
 $Comp
-L Device:R R?
+L Device:R R5
 U 1 1 606373DA
 P 5100 3575
-F 0 "R?" H 5170 3621 50  0000 L CNN
+F 0 "R5" H 5170 3621 50  0000 L CNN
 F 1 "3.3k" H 5170 3530 50  0000 L CNN
 F 2 "" V 5030 3575 50  0001 C CNN
@@
 	5100 2775 5100 3425
 $Comp
-L power:GND #PWR?
+L power:GND #PWR09
 U 1 1 6063EA65
 P 5100 3800
-F 0 "#PWR?" H 5100 3550 50  0001 C CNN
+F 0 "#PWR09" H 5100 3550 50  0001 C CNN
 F 1 "GND" H 5105 3627 50  0000 C CNN
 F 2 "" H 5100 3800 50  0001 C CNN
@@
 	5100 3800 5100 3725
 $Comp
-L Device:C C?
+L Device:C C40
 U 1 1 6064A39B
 P 9300 2050
-F 0 "C?" H 9415 2096 50  0000 L CNN
+F 0 "C40" H 9415 2096 50  0000 L CNN
 F 1 "1u" H 9415 2005 50  0000 L CNN
 F 2 "" H 9338 1900 50  0001 C CNN
@@
 $EndComp
 $Comp
-L Device:C C?
+L Device:C C42
 U 1 1 6064B02C
 P 9750 2050
-F 0 "C?" H 9865 2096 50  0000 L CNN
+F 0 "C42" H 9865 2096 50  0000 L CNN
 F 1 "47p" H 9865 2005 50  0000 L CNN
 F 2 "" H 9788 1900 50  0001 C CNN
@@
 $EndComp
 $Comp
-L Device:C C?
+L Device:C C43
 U 1 1 6065065E
 P 10175 2050
-F 0 "C?" H 10290 2096 50  0000 L CNN
+F 0 "C43" H 10290 2096 50  0000 L CNN
 F 1 "1n" H 10290 2005 50  0000 L CNN
 F 2 "" H 10213 1900 50  0001 C CNN
@@
 	9300 1750 9750 1750
 $Comp
-L power:GND #PWR?
+L power:GND #PWR038
 U 1 1 60667EF4
 P 9300 2200
-F 0 "#PWR?" H 9300 1950 50  0001 C CNN
+F 0 "#PWR038" H 9300 1950 50  0001 C CNN
 F 1 "GND" H 9305 2027 50  0000 C CNN
 F 2 "" H 9300 2200 50  0001 C CNN
@@
 $EndComp
 $Comp
-L power:GND #PWR?
+L power:GND #PWR039
 U 1 1 60668416
 P 9750 2200
-F 0 "#PWR?" H 9750 1950 50  0001 C CNN
+F 0 "#PWR039" H 9750 1950 50  0001 C CNN
 F 1 "GND" H 9755 2027 50  0000 C CNN
 F 2 "" H 9750 2200 50  0001 C CNN
@@
 $EndComp
 $Comp
-L power:GND #PWR?
+L power:GND #PWR040
 U 1 1 60668A00
 P 10175 2200
-F 0 "#PWR?" H 10175 1950 50  0001 C CNN
+F 0 "#PWR040" H 10175 1950 50  0001 C CNN
 F 1 "GND" H 10180 2027 50  0000 C CNN
 F 2 "" H 10175 2200 50  0001 C CNN
@@
 $EndComp
 $Comp
-L Device:L L?
+L Device:L L8
 U 1 1 606892C0
 P 7675 2100
-F 0 "L?" H 7727 2146 50  0000 L CNN
+F 0 "L8" H 7727 2146 50  0000 L CNN
 F 1 "22n" H 7727 2055 50  0000 L CNN
 F 2 "" H 7675 2100 50  0001 C CNN
@@
 	7675 1750 9300 1750
 $Comp
-L Device:L L?
+L Device:L L5
 U 1 1 606FF9FC
 P 3750 3275
-F 0 "L?" V 3940 3275 50  0000 C CNN
+F 0 "L5" V 3940 3275 50  0000 C CNN
 F 1 "10n" V 3849 3275 50  0000 C CNN
 F 2 "" H 3750 3275 50  0001 C CNN

Commit message: Lots of work on routing and pcb layout
Parts:
- removed FL1: B39871B4316P810, Filter:Filter_1109-5_1.1x0.9mm, symbol Filter:B39162B8813P810
- added FL1: SAW_RF_filterB3725, TU-HW RF LIB:SON120P300X300X110-6N, symbol TU-rescue:SAW_RF_filterB3725-B39871B3725U410
- C11: value 220n -> 220p
- C12, C14, C15, C16, C18, C38, C40, C42, C43: footprint (none) -> Capacitor_SMD:C_0603_1608Metric
- C7: value 0 -> DNM
- IC1: footprint QFN65P400X400X100-17N -> Package_DFN_QFN:QFN-16-1EP_4x4mm_P0.65mm_EP2.15x2.15mm
- L4, L5, L6, L7, L8, L9: footprint (none) -> Inductor_SMD:L_0603_1608Metric
- R11, R12, R4, R5, R9: footprint (none) -> Resistor_SMD:R_0603_1608Metric
- TP1: footprint (none) -> TestPoint:TestPoint_Pad_2.0x2.0mm
Changed lines of the file:
@@
 	2000 2825 1650 2825
-Wire Wire Line
-	2600 3275 2450 3275
-Connection ~ 2600 3275
-Wire Wire Line
-	2600 2825 2600 3275
 Wire Wire Line
 	2300 2825 2600 2825
@@
 L power:GND #PWR013
 U 1 1 601F291A
-P 2150 3775
-F 0 "#PWR013" H 2150 3525 50  0001 C CNN
-F 1 "GND" H 2155 3602 50  0000 C CNN
-F 2 "" H 2150 3775 50  0001 C CNN
-F 3 "" H 2150 3775 50  0001 C CNN
-	1    2150 3775
+P 2150 3675
+F 0 "#PWR013" H 2150 3425 50  0001 C CNN
+F 1 "GND" H 2155 3502 50  0000 C CNN
+F 2 "" H 2150 3675 50  0001 C CNN
+F 3 "" H 2150 3675 50  0001 C CNN
+	1    2150 3675
 	-1   0    0    -1
 $EndComp
 Wire Wire Line
-	2150 3675 1850 3675
-Connection ~ 2150 3675
-Wire Wire Line
-	2150 3675 2150 3775
-Wire Wire Line
-	1850 3675 1850 3475
-Wire Wire Line
-	2450 3675 2150 3675
-Wire Wire Line
-	2450 3475 2450 3675
-Wire Wire Line
-	3250 3275 2600 3275
-$Comp
-L Filter:B39162B8813P810 FL1
-U 1 1 601EC5BA
-P 2150 3375
-F 0 "FL1" H 2150 3742 50  0000 C CNN
-F 1 "B39871B4316P810" H 2150 3651 50  0000 C CNN
-F 2 "Filter:Filter_1109-5_1.1x0.9mm" H 2150 3375 50  0001 C CNN
-F 3 "https://www.digikey.se/product-detail/en/qualcomm-rf360-a-qualcomm-tdk-joint-venture/B39871B4316P810/B39871B4316P810CT-ND/8737775" H 2080 3405 50  0001 C CNN
-	1    2150 3375
-	-1   0    0    -1
-$EndComp
+	2150 3575 2150 3675
 Wire Wire Line
 	3250 3275 3250 3375
@@
 F 0 "R9" H 5555 7054 50  0000 R CNN
 F 1 "10k" H 5555 7145 50  0000 R CNN
-F 2 "" V 5555 7100 50  0001 C CNN
+F 2 "Resistor_SMD:R_0603_1608Metric" V 5555 7100 50  0001 C CNN
 F 3 "~" H 5625 7100 50  0001 C CNN
 	1    5625 7100
@@
 F 0 "R11" H 5830 7054 50  0000 R CNN
 F 1 "10k" H 5830 7145 50  0000 R CNN
-F 2 "" V 5830 7100 50  0001 C CNN
+F 2 "Resistor_SMD:R_0603_1608Metric" V 5830 7100 50  0001 C CNN
 F 3 "~" H 5900 7100 50  0001 C CNN
 	1    5900 7100
@@
 F 0 "R12" H 6130 7054 50  0000 R CNN
 F 1 "10k" H 6130 7145 50  0000 R CNN
-F 2 "" V 6130 7100 50  0001 C CNN
+F 2 "Resistor_SMD:R_0603_1608Metric" V 6130 7100 50  0001 C CNN
 F 3 "~" H 6200 7100 50  0001 C CNN
 	1    6200 7100
@@
 F 0 "TP1" V 4079 1163 50  0000 L CNN
 F 1 "VDD_CC1190" V 4170 1163 50  0000 L CNN
-F 2 "" H 4325 975 50  0001 C CNN
+F 2 "TestPoint:TestPoint_Pad_2.0x2.0mm" H 4325 975 50  0001 C CNN
 F 3 "~" H 4325 975 50  0001 C CNN
 	1    4125 975
@@
 P 1800 1225
 F 0 "C11" H 1915 1271 50  0000 L CNN
-F 1 "220n" H 1915 1180 50  0000 L CNN
+F 1 "220p" H 1915 1180 50  0000 L CNN
 F 2 "Capacitor_SMD:C_0603_1608Metric" H 1838 1075 50  0001 C CNN
 F 3 "~" H 1800 1225 50  0001 C CNN
@@
 F 0 "L4" V 3940 1750 50  0000 C CNN
 F 1 "L" V 3849 1750 50  0000 C CNN
-F 2 "" H 3750 1750 50  0001 C CNN
+F 2 "Inductor_SMD:L_0603_1608Metric" H 3750 1750 50  0001 C CNN
 F 3 "~" H 3750 1750 50  0001 C CNN
 	1    3750 1750
@@
 P 4000 5250
 F 0 "C7" H 4115 5296 50  0000 L CNN
-F 1 "0" H 4115 5205 50  0000 L CNN
+F 1 "DNM" H 4115 5205 50  0000 L CNN
 F 2 "Capacitor_SMD:C_0603_1608Metric" H 4038 5100 50  0001 C CNN
 F 3 "~" H 4000 5250 50  0001 C CNN
@@
 F 0 "IC1" H 6050 3340 50  0000 C CNN
 F 1 "CC1190" H 6050 3249 50  0000 C CNN
-F 2 "QFN65P400X400X100-17N" H 5750 3375 50  0001 L BNN
+F 2 "Package_DFN_QFN:QFN-16-1EP_4x4mm_P0.65mm_EP2.15x2.15mm" H 5750 3375 50  0001 L BNN
 F 3 "" H 6450 3475 50  0001 L BNN
 	1    6250 2775
@@
 F 0 "L7" H 6277 5346 50  0000 L CNN
 F 1 "7.5n" H 6277 5255 50  0000 L CNN
-F 2 "" H 6225 5300 50  0001 C CNN
+F 2 "Inductor_SMD:L_0603_1608Metric" H 6225 5300 50  0001 C CNN
 F 3 "~" H 6225 5300 50  0001 C CNN
 	1    6225 5300
@@
 F 0 "C15" H 6340 5721 50  0000 L CNN
 F 1 "12p" H 6340 5630 50  0000 L CNN
-F 2 "" H 6263 5525 50  0001 C CNN
+F 2 "Capacitor_SMD:C_0603_1608Metric" H 6263 5525 50  0001 C CNN
 F 3 "~" H 6225 5675 50  0001 C CNN
 	1    6225 5675
@@
 F 0 "C18" V 7823 6050 50  0000 C CNN
 F 1 "12p" V 7914 6050 50  0000 C CNN
-F 2 "" H 8113 5900 50  0001 C CNN
+F 2 "Capacitor_SMD:C_0603_1608Metric" H 8113 5900 50  0001 C CNN
 F 3 "~" H 8075 6050 50  0001 C CNN
 	1    8075 6050
@@
 F 0 "C16" V 6598 4950 50  0000 C CNN
 F 1 "47p" V 6689 4950 50  0000 C CNN
-F 2 "" H 6888 4800 50  0001 C CNN
+F 2 "Capacitor_SMD:C_0603_1608Metric" H 6888 4800 50  0001 C CNN
 F 3 "~" H 6850 4950 50  0001 C CNN
 	1    6850 4950
@@
 F 0 "L9" H 8602 2721 50  0000 L CNN
 F 1 "2.7n" H 8602 2630 50  0000 L CNN
-F 2 "" H 8550 2675 50  0001 C CNN
+F 2 "Inductor_SMD:L_0603_1608Metric" H 8550 2675 50  0001 C CNN
 F 3 "~" H 8550 2675 50  0001 C CNN
 	1    8550 2675
@@
 F 0 "C38" H 8665 3121 50  0000 L CNN
 F 1 "2.7p" H 8665 3030 50  0000 L CNN
-F 2 "" H 8588 2925 50  0001 C CNN
+F 2 "Capacitor_SMD:C_0603_1608Metric" H 8588 2925 50  0001 C CNN
 F 3 "~" H 8550 3075 50  0001 C CNN
 	1    8550 3075
@@
 F 0 "C12" H 3590 2046 50  0000 L CNN
 F 1 "15p" H 3590 1955 50  0000 L CNN
-F 2 "" H 3513 1850 50  0001 C CNN
+F 2 "Capacitor_SMD:C_0603_1608Metric" H 3513 1850 50  0001 C CNN
 F 3 "~" H 3475 2000 50  0001 C CNN
 	1    3475 2000
@@
 F 0 "C14" H 4365 2046 50  0000 L CNN
 F 1 "27p" H 4365 1955 50  0000 L CNN
-F 2 "" H 4288 1850 50  0001 C CNN
+F 2 "Capacitor_SMD:C_0603_1608Metric" H 4288 1850 50  0001 C CNN
 F 3 "~" H 4250 2000 50  0001 C CNN
 	1    4250 2000
@@
 F 0 "L6" H 5102 2221 50  0000 L CNN
 F 1 "15n" H 5102 2130 50  0000 L CNN
-F 2 "" H 5050 2175 50  0001 C CNN
+F 2 "Inductor_SMD:L_0603_1608Metric" H 5050 2175 50  0001 C CNN
 F 3 "~" H 5050 2175 50  0001 C CNN
 	1    5050 2175
@@
 F 0 "R4" H 4820 2221 50  0000 L CNN
 F 1 "47" H 4820 2130 50  0000 L CNN
-F 2 "" V 4680 2175 50  0001 C CNN
+F 2 "Resistor_SMD:R_0603_1608Metric" V 4680 2175 50  0001 C CNN
 F 3 "~" H 4750 2175 50  0001 C CNN
 	1    4750 2175
@@
 F 0 "R5" H 5170 3621 50  0000 L CNN
 F 1 "3.3k" H 5170 3530 50  0000 L CNN
-F 2 "" V 5030 3575 50  0001 C CNN
+F 2 "Resistor_SMD:R_0603_1608Metric" V 5030 3575 50  0001 C CNN
 F 3 "~" H 5100 3575 50  0001 C CNN
 	1    5100 3575
@@
 F 0 "C40" H 9415 2096 50  0000 L CNN
 F 1 "1u" H 9415 2005 50  0000 L CNN
-F 2 "" H 9338 1900 50  0001 C CNN
+F 2 "Capacitor_SMD:C_0603_1608Metric" H 9338 1900 50  0001 C CNN
 F 3 "~" H 9300 2050 50  0001 C CNN
 	1    9300 2050
@@
 F 0 "C42" H 9865 2096 50  0000 L CNN
 F 1 "47p" H 9865 2005 50  0000 L CNN
-F 2 "" H 9788 1900 50  0001 C CNN
+F 2 "Capacitor_SMD:C_0603_1608Metric" H 9788 1900 50  0001 C CNN
 F 3 "~" H 9750 2050 50  0001 C CNN
 	1    9750 2050
@@
 F 0 "C43" H 10290 2096 50  0000 L CNN
 F 1 "1n" H 10290 2005 50  0000 L CNN
-F 2 "" H 10213 1900 50  0001 C CNN
+F 2 "Capacitor_SMD:C_0603_1608Metric" H 10213 1900 50  0001 C CNN
 F 3 "~" H 10175 2050 50  0001 C CNN
 	1    10175 2050
@@
 F 0 "L8" H 7727 2146 50  0000 L CNN
 F 1 "22n" H 7727 2055 50  0000 L CNN
-F 2 "" H 7675 2100 50  0001 C CNN
+F 2 "Inductor_SMD:L_0603_1608Metric" H 7675 2100 50  0001 C CNN
 F 3 "~" H 7675 2100 50  0001 C CNN
 	1    7675 2100
@@
 F 0 "L5" V 3940 3275 50  0000 C CNN
 F 1 "10n" V 3849 3275 50  0000 C CNN
-F 2 "" H 3750 3275 50  0001 C CNN
+F 2 "Inductor_SMD:L_0603_1608Metric" H 3750 3275 50  0001 C CNN
 F 3 "~" H 3750 3275 50  0001 C CNN
 	1    3750 3275
@@
 Wire Wire Line
 	3600 3275 3250 3275
-Connection ~ 3250 3275
 Wire Wire Line
 	3900 3275 5350 3275
@@
 	2400 975  4000 975
 Connection ~ 4000 975
+$Comp
+L TU-rescue:SAW_RF_filterB3725-B39871B3725U410 FL1
+U 1 1 6035BDD1
+P 2150 3275
+AR Path="/6035BDD1" Ref="FL1"  Part="1"
+AR Path="/6014566F/6035BDD1" Ref="FL1"  Part="1"
+F 0 "FL1" H 2150 3642 50  0000 C CNN
+F 1 "SAW_RF_filterB3725" H 2150 3551 50  0000 C CNN
+F 2 "TU-HW RF LIB:SON120P300X300X110-6N" H 2150 3625 50  0001 C CNN
+F 3 "https://product.tdk.com/search-template/en/documents/data_sheet/40/ds/mc/B9482.pdf" H 2080 3305 50  0001 C CNN
+	1    2150 3275
+	1    0    0    -1
+$EndComp
+Connection ~ 2100 3575
+Wire Wire Line
+	2100 3575 2000 3575
+Connection ~ 2200 3575
+Wire Wire Line
+	2200 3575 2150 3575
+Wire Wire Line
+	2200 3575 2300 3575
+Connection ~ 2150 3575
+Wire Wire Line
+	2150 3575 2100 3575
+Connection ~ 3250 3275
+Wire Wire Line
+	3250 3275 2600 3275
+Wire Wire Line
+	2600 2825 2600 3275
+Connection ~ 2600 3275
+Wire Wire Line
+	2600 3275 2450 3275
 $EndSCHEMATC

Commit message: More routing changes
Connections:
- wire segments 107 -> 104
Other:
- moved on the sheet: R11, R12, R9
Changed lines of the file:
@@
 	-1   0    0    -1
 $EndComp
-Text HLabel 6475 7325 2    59   Input ~ 0
+Text HLabel 7875 3500 2    59   Input ~ 0
 PA_EN
-Text Label 5125 6500 0    59   ~ 0
-PA_EN
-Text Label 5125 6600 0    59   ~ 0
-LNA_EN
-Text Label 5125 6700 0    59   ~ 0
+Text HLabel 7875 3700 2    59   Input ~ 0
 HGM
-Text HLabel 6475 7525 2    59   Input ~ 0
-HGM
-Text HLabel 6475 7425 2    59   Input ~ 0
+Text HLabel 7875 3600 2    59   Input ~ 0
 LNA_EN
 $Comp
 L Device:R R9
 U 1 1 6051AA9E
-P 5625 7100
-F 0 "R9" H 5555 7054 50  0000 R CNN
-F 1 "10k" H 5555 7145 50  0000 R CNN
-F 2 "Resistor_SMD:R_0603_1608Metric" V 5555 7100 50  0001 C CNN
-F 3 "~" H 5625 7100 50  0001 C CNN
-	1    5625 7100
+P 6875 3275
+F 0 "R9" H 6805 3229 50  0000 R CNN
+F 1 "10k" H 6805 3320 50  0000 R CNN
+F 2 "Resistor_SMD:R_0603_1608Metric" V 6805 3275 50  0001 C CNN
+F 3 "~" H 6875 3275 50  0001 C CNN
+	1    6875 3275
 	-1   0    0    1
 $EndComp
@@
 L Device:R R11
 U 1 1 6051F9F3
-P 5900 7100
-F 0 "R11" H 5830 7054 50  0000 R CNN
-F 1 "10k" H 5830 7145 50  0000 R CNN
-F 2 "Resistor_SMD:R_0603_1608Metric" V 5830 7100 50  0001 C CNN
-F 3 "~" H 5900 7100 50  0001 C CNN
-	1    5900 7100
+P 7150 3275
+F 0 "R11" H 7080 3229 50  0000 R CNN
+F 1 "10k" H 7080 3320 50  0000 R CNN
+F 2 "Resistor_SMD:R_0603_1608Metric" V 7080 3275 50  0001 C CNN
+F 3 "~" H 7150 3275 50  0001 C CNN
+	1    7150 3275
 	-1   0    0    1
 $EndComp
@@
 L Device:R R12
 U 1 1 6052394F
-P 6200 7100
-F 0 "R12" H 6130 7054 50  0000 R CNN
-F 1 "10k" H 6130 7145 50  0000 R CNN
-F 2 "Resistor_SMD:R_0603_1608Metric" V 6130 7100 50  0001 C CNN
-F 3 "~" H 6200 7100 50  0001 C CNN
-	1    6200 7100
+P 7450 3275
+F 0 "R12" H 7380 3229 50  0000 R CNN
+F 1 "10k" H 7380 3320 50  0000 R CNN
+F 2 "Resistor_SMD:R_0603_1608Metric" V 7380 3275 50  0001 C CNN
+F 3 "~" H 7450 3275 50  0001 C CNN
+	1    7450 3275
 	-1   0    0    1
 $EndComp
 Wire Wire Line
-	6475 7325 6200 7325
-Wire Wire Line
-	6200 7325 6200 7250
-Wire Wire Line
-	6475 7425 5900 7425
-Wire Wire Line
-	5900 7425 5900 7250
-Wire Wire Line
-	6475 7525 5625 7525
-Wire Wire Line
-	5625 7525 5625 7250
-Wire Wire Line
-	5625 6950 5625 6700
-Wire Wire Line
-	5125 6700 5625 6700
-Wire Wire Line
-	5900 6600 5900 6950
-Wire Wire Line
-	6200 6950 6200 6500
-Wire Wire Line
-	5125 6500 6200 6500
-Wire Wire Line
-	5125 6600 5900 6600
+	7450 3500 7450 3425
+Wire Wire Line
+	7150 3600 7150 3425
+Wire Wire Line
+	6875 3700 6875 3425
 $Comp
 L Connector:TestPoint TP1
@@
 Wire Wire Line
 	8325 6050 8325 2675
-Wire Wire Line
-	8325 2675 6750 2675
 $Comp
 L Device:C C16
@@
 Wire Wire Line
 	7000 4950 7675 4950
-Text Label 7100 2775 2    59   ~ 0
-HGM
-Text Label 7100 2875 2    59   ~ 0
-LNA_EN
-Text Label 7100 2975 2    59   ~ 0
-PA_EN
-Wire Wire Line
-	6750 2775 7100 2775
-Wire Wire Line
-	6750 2875 7100 2875
-Wire Wire Line
-	6750 2975 7100 2975
 Wire Wire Line
 	3225 2975 5350 2975
@@
 Wire Wire Line
 	2600 3275 2450 3275
+Wire Wire Line
+	6750 2675 8325 2675
+Wire Wire Line
+	6875 3125 6875 2975
+Wire Wire Line
+	6875 2975 6750 2975
+Wire Wire Line
+	6750 2875 7150 2875
+Wire Wire Line
+	7150 2875 7150 3125
+Wire Wire Line
+	7450 3125 7450 2775
+Wire Wire Line
+	7450 2775 6750 2775
+Wire Wire Line
+	7450 3500 7875 3500
+Wire Wire Line
+	7150 3600 7875 3600
+Wire Wire Line
+	6875 3700 7875 3700
 $EndSCHEMATC

Commit message: Added mounting holes and terminal block
Parts:
- removed FL1: SAW_RF_filterB3725, TU-HW RF LIB:SON120P300X300X110-6N, symbol TU-rescue:SAW_RF_filterB3725-B39871B3725U410
- added FL1: SAW_RF_filterB3725, TU-HW RF LIB:SON120P300X300X110-6N, symbol B39871B3725U410:SAW_RF_filterB3725
Connections:
- net labels added: RFIO
- net labels removed: CC1190_RFIO
- wire segments 104 -> 105
