File: MCU.sch (KiCad schematic (older format))
At the start: 0 parts

Commit message: Started work on CC1200
might not be actual final tranciever
Changed lines of the file:
@@
 $Descr A4 11693 8268
 encoding utf-8
-Sheet 3 6
+Sheet 2 6
 Title ""
 Date ""
@@
 MISO
 Text HLabel 8300 3300 2    59   Output ~ 0
-~SS
+~CS
 $EndSCHEMATC

Commit message: Started work on MCU
Parts:
- added C33, C34, C35, C37, C38, C39, C41, C42, C43, C45, C46, C47, C49, C50, C51, C52, C53: 100n, symbol Device:C
- added C36, C40, C44: 1u, symbol Device:C
- added C48, C?: C, symbol Device:C
- added C54: 4.7u, symbol Device:C
- added D? (x3): LED, symbol Device:LED
- added J?: ARM_JTAG_SWD_10, symbol KTHFS:ARM_JTAG_SWD_10
- added R? (x4): 10k, symbol Device:R
- added R? (x3): R, symbol Device:R
- added U5: STM32F769IITx, Package_QFP:LQFP-176_24x24mm_P0.5mm, symbol MCU_ST_STM32F7:STM32F769IITx
Connections:
- new net: D?.2 (A), R?.2 (x3)
- new net +3V3: C33.1, C34.1, C35.1, C36.1, C37.1, C38.1, C39.1, C40.1, C41.1, C42.1, C43.1, C44.1, C45.1, C47.1, C49.1, C50.1, C51.1, C52.1, C53.1, C54.1, J?.1 (VTref), R?.1, R?.2, U5.106 (VDD12DSI), U5.118 (VDDUSB), U5.131 (VDD), U5.136 (VDD), U5.149 (VDDSDMMC), U5.15 (VDD), U5.159 (VDD), U5.172 (VDD), U5.23 (VDD), U5.36 (VDD), U5.39 (VDDA), U5.49 (VDD), U5.6 (VBAT), U5.62 (VDD), U5.72 (VDD), U5.82 (VDD), U5.96 (VDD), U5.99 (VDDDSI)
- new net BOOT0: R?.2
- new net BYPASS_REG: R?.1
- new net CAP_1: C46.1
- new net CAP_2: C48.1
- new net GND: C33.2, C34.2, C35.2, C36.2, C37.2, C38.2, C39.2, C40.2, C41.2, C42.2, C43.2, C44.2, C45.2, C46.2, C47.2, C48.2, C49.2, C50.2, C51.2, C52.2, C53.2, C54.2, C?.2, D?.1 (K), D?.1 (K), D?.1 (K), J?.3 (GND), J?.5 (GND), J?.9 (GNDDetect), R?.1, R?.2, U5.103 (VSSDSI), U5.109 (VSSDSI), U5.117 (VSS), U5.130 (VSS), U5.135 (VSS), U5.14 (VSS), U5.148 (VSS), U5.158 (VSS), U5.22 (VSS), U5.37 (VSSA), U5.61 (VSS), U5.71 (VSS), U5.95 (VSS)
- new net LED_1: R?.1
- new net LED_2: R?.1
- new net LED_3: R?.1
- new net NRST: C?.1, J?.10 (~RESET~), R?.1
- new net PDR_ON: R?.2
- new net SWCLK: J?.4 (SWDCLK/TCK), U5.128 (PA13)
- new net SWDIO: J?.2 (SWDIO/TMS), U5.137 (PA14)
Other:
- note added: "Bootloader connector\n"
- note added: "Configuration pins\n"
- note added: "Debug leds\n"
- note added: "USE CAN1/CAN2 and CAN3"
- note added: "USE SPI1,4,5,6 for 54 Mbps"
- note added: "VDDA\n"
- note added: "VDDSDMMCC"
- note added: "VDDUSB"
- note added: "VDD\n"
- note added: "Vcap\n"

Commit message: More work on tranciever and PA
Parts:
- gave numbers to parts that had none: 12
Changed lines of the file:
@@
 $Descr A3 16535 11693
 encoding utf-8
-Sheet 2 6
+Sheet 5 6
 Title ""
 Date ""
@@
 $EndComp
 $Comp
-L KTHFS:ARM_JTAG_SWD_10 J?
+L KTHFS:ARM_JTAG_SWD_10 J5
 U 1 1 601E65F6
 P 14500 5050
-F 0 "J?" H 14550 6200 50  0000 R CNN
+F 0 "J5" H 14550 6200 50  0000 R CNN
 F 1 "ARM_JTAG_SWD_10" H 14850 6100 50  0000 R CNN
 F 2 "" H 14500 5050 50  0001 C CNN
@@
 	14500 4400 14500 4350
 $Comp
-L power:+3.3V #PWR?
+L power:+3.3V #PWR052
 U 1 1 601F3500
 P 14500 4350
-F 0 "#PWR?" H 14500 4200 50  0001 C CNN
+F 0 "#PWR052" H 14500 4200 50  0001 C CNN
 F 1 "+3.3V" H 14515 4523 50  0000 C CNN
 F 2 "" H 14500 4350 50  0001 C CNN
@@
 $EndComp
 $Comp
-L power:GND #PWR?
+L power:GND #PWR053
 U 1 1 601F4213
 P 14500 5700
-F 0 "#PWR?" H 14500 5450 50  0001 C CNN
+F 0 "#PWR053" H 14500 5450 50  0001 C CNN
 F 1 "GND" H 14505 5527 50  0000 C CNN
 F 2 "" H 14500 5700 50  0001 C CNN
@@
 BYPASS_REG
 $Comp
-L Device:R R?
+L Device:R R11
 U 1 1 601FD9AC
 P 14650 8500
-F 0 "R?" V 14857 8500 50  0000 C CNN
+F 0 "R11" V 14857 8500 50  0000 C CNN
 F 1 "10k" V 14766 8500 50  0000 C CNN
 F 2 "" V 14580 8500 50  0001 C CNN
@@
 $EndComp
 $Comp
-L Device:R R?
+L Device:R R12
 U 1 1 601FE255
 P 14650 8850
-F 0 "R?" V 14443 8850 50  0000 C CNN
+F 0 "R12" V 14443 8850 50  0000 C CNN
 F 1 "10k" V 14534 8850 50  0000 C CNN
 F 2 "" V 14580 8850 50  0001 C CNN
@@
 	14350 8850 14350 9100
 $Comp
-L power:GND #PWR?
+L power:GND #PWR051
 U 1 1 602079EB
 P 14350 9100
-F 0 "#PWR?" H 14350 8850 50  0001 C CNN
+F 0 "#PWR051" H 14350 8850 50  0001 C CNN
 F 1 "GND" H 14355 8927 50  0000 C CNN
 F 2 "" H 14350 9100 50  0001 C CNN
@@
 NRST
 $Comp
-L Device:C C?
+L Device:C C56
 U 1 1 6020C680
 P 15050 7800
-F 0 "C?" H 15165 7846 50  0000 L CNN
+F 0 "C56" H 15165 7846 50  0000 L CNN
 F 1 "C" H 15165 7755 50  0000 L CNN
 F 2 "" H 15088 7650 50  0001 C CNN
@@
 	15050 7650 15400 7650
 $Comp
-L power:GND #PWR?
+L power:GND #PWR054
 U 1 1 6020E0D9
 P 15050 7950
-F 0 "#PWR?" H 15050 7700 50  0001 C CNN
+F 0 "#PWR054" H 15050 7700 50  0001 C CNN
 F 1 "GND" H 15055 7777 50  0000 C CNN
 F 2 "" H 15050 7950 50  0001 C CNN
@@
 Connection ~ 14300 7300
 $Comp
-L power:+3.3V #PWR?
+L power:+3.3V #PWR050
 U 1 1 60212469
 P 14300 7200
-F 0 "#PWR?" H 14300 7050 50  0001 C CNN
+F 0 "#PWR050" H 14300 7050 50  0001 C CNN
 F 1 "+3.3V" H 14315 7373 50  0000 C CNN
 F 2 "" H 14300 7200 50  0001 C CNN
@@
 $EndComp
 $Comp
-L Device:R R?
+L Device:R R9
 U 1 1 602177C3
 P 14650 7300
-F 0 "R?" V 14857 7300 50  0000 C CNN
+F 0 "R9" V 14857 7300 50  0000 C CNN
 F 1 "10k" V 14766 7300 50  0000 C CNN
 F 2 "" V 14580 7300 50  0001 C CNN
@@
 $EndComp
 $Comp
-L Device:R R?
+L Device:R R10
 U 1 1 602177C9
 P 14650 7650
-F 0 "R?" V 14443 7650 50  0000 C CNN
+F 0 "R10" V 14443 7650 50  0000 C CNN
 F 1 "10k" V 14534 7650 50  0000 C CNN
 F 2 "" V 14580 7650 50  0001 C CNN
@@
 	3650 10050 3750 10050
 $Comp
-L power:GND #PWR?
+L power:GND #PWR05
 U 1 1 6021C6BB
 P 3750 10150
-F 0 "#PWR?" H 3750 9900 50  0001 C CNN
+F 0 "#PWR05" H 3750 9900 50  0001 C CNN
 F 1 "GND" H 3755 9977 50  0000 C CNN
 F 2 "" H 3750 10150 50  0001 C CNN
@@
 	3950 1150 4050 1150
 $Comp
-L power:+3.3V #PWR?
+L power:+3.3V #PWR046
 U 1 1 6021FE33
 P 4050 1050
-F 0 "#PWR?" H 4050 900 50  0001 C CNN
+F 0 "#PWR046" H 4050 900 50  0001 C CNN
 F 1 "+3.3V" H 4065 1223 50  0000 C CNN
 F 2 "" H 4050 1050 50  0001 C CNN
@@
 Debug leds\n
 $Comp
-L Device:R R?
+L Device:R R1
 U 1 1 602896BD
 P 12550 7350
-F 0 "R?" V 12757 7350 50  0000 C CNN
+F 0 "R1" V 12757 7350 50  0000 C CNN
 F 1 "R" V 12666 7350 50  0000 C CNN
 F 2 "" V 12480 7350 50  0001 C CNN
@@
 $EndComp
 $Comp
-L Device:LED D?
+L Device:LED D1
 U 1 1 6028A414
 P 12850 7350
-F 0 "D?" H 12843 7095 50  0000 C CNN
+F 0 "D1" H 12843 7095 50  0000 C CNN
 F 1 "LED" H 12843 7186 50  0000 C CNN
 F 2 "" H 12850 7350 50  0001 C CNN
@@
 LED_3
 $Comp
-L Device:R R?
+L Device:R R2
 U 1 1 602A59D1
 P 12550 8050
-F 0 "R?" V 12757 8050 50  0000 C CNN
+F 0 "R2" V 12757 8050 50  0000 C CNN
 F 1 "R" V 12666 8050 50  0000 C CNN
 F 2 "" V 12480 8050 50  0001 C CNN
@@
 $EndComp
 $Comp
-L Device:LED D?
+L Device:LED D2
 U 1 1 602A59D7
 P 12850 8050
-F 0 "D?" H 12843 7795 50  0000 C CNN
+F 0 "D2" H 12843 7795 50  0000 C CNN
 F 1 "LED" H 12843 7886 50  0000 C CNN
 F 2 "" H 12850 8050 50  0001 C CNN
@@
 	12100 8050 12400 8050
 $Comp
-L Device:R R?
+L Device:R R8
 U 1 1 602AA1DC
 P 12550 8750
-F 0 "R?" V 12757 8750 50  0000 C CNN
+F 0 "R8" V 12757 8750 50  0000 C CNN
 F 1 "R" V 12666 8750 50  0000 C CNN
 F 2 "" V 12480 8750 50  0001 C CNN
@@
 $EndComp
 $Comp
-L Device:LED D?
+L Device:LED D7
 U 1 1 602AA1E2
 P 12850 8750
-F 0 "D?" H 12843 8495 50  0000 C CNN
+F 0 "D7" H 12843 8495 50  0000 C CNN
 F 1 "LED" H 12843 8586 50  0000 C CNN
 F 2 "" H 12850 8750 50  0001 C CNN
@@
 	12100 8750 12400 8750
 $Comp
-L power:GND #PWR?
+L power:GND #PWR047
 U 1 1 602B702D
 P 13100 7500
-F 0 "#PWR?" H 13100 7250 50  0001 C CNN
+F 0 "#PWR047" H 13100 7250 50  0001 C CNN
 F 1 "GND" H 13105 7327 50  0000 C CNN
 F 2 "" H 13100 7500 50  0001 C CNN
@@
 $EndComp
 $Comp
-L power:GND #PWR?
+L power:GND #PWR048
 U 1 1 602B7904
 P 13100 8200
-F 0 "#PWR?" H 13100 7950 50  0001 C CNN
+F 0 "#PWR048" H 13100 7950 50  0001 C CNN
 F 1 "GND" H 13105 8027 50  0000 C CNN
 F 2 "" H 13100 8200 50  0001 C CNN
@@
 $EndComp
 $Comp
-L power:GND #PWR?
+L power:GND #PWR049
 U 1 1 602B7A6F
 P 13100 8900
-F 0 "#PWR?" H 13100 8650 50  0001 C CNN
+F 0 "#PWR049" H 13100 8650 50  0001 C CNN
 F 1 "GND" H 13105 8727 50  0000 C CNN
 F 2 "" H 13100 8900 50  0001 C CNN
@@
 Wire Notes Line
 	13400 9450 13400 6850
+Text HLabel 6900 6300 2    59   Output ~ 0
+HGM
+Text HLabel 6900 6400 2    59   Output ~ 0
+LNA_EN
+Text HLabel 6900 6500 2    59   Output ~ 0
+PA_EN
+Text HLabel 6900 6950 2    59   BiDi ~ 0
+RF_GPIO0
+Text HLabel 6900 6850 2    59   BiDi ~ 0
+RF_GPIO2
+Text HLabel 6900 6750 2    59   BiDi ~ 0
+RF_GPIO3
 $EndSCHEMATC

Commit message: Small changes to schematic
Connections:
- net SWDIO: no longer U5.137 (PA14)
Changed lines of the file:
@@
 $Descr A3 16535 11693
 encoding utf-8
-Sheet 5 6
+Sheet 4 6
 Title ""
 Date ""
@@
 Comment4 ""
 $EndDescr
-Text HLabel 6900 5750 2    59   Output ~ 0
+Text HLabel 5400 4250 2    59   Output ~ 0
 SLCK
-Text HLabel 6900 5850 2    59   Output ~ 0
+Text HLabel 5400 4350 2    59   Output ~ 0
 MOSI
-Text HLabel 6900 5950 2    59   Input ~ 0
+Text HLabel 5400 4450 2    59   Input ~ 0
 MISO
-Text HLabel 6900 6050 2    59   Output ~ 0
+Text HLabel 5400 4550 2    59   Output ~ 0
 ~CS
 $Comp
@@
 	1    0    0    -1
 $EndComp
-Text HLabel 6900 4650 2    50   Input ~ 0
+Text HLabel 5400 3150 2    50   Input ~ 0
 CAN_TX_1
-Text HLabel 6900 4750 2    50   Output ~ 0
+Text HLabel 5400 3250 2    50   Output ~ 0
 CAN_RX_1
-Text HLabel 6900 4950 2    50   Input ~ 0
+Text HLabel 5400 3450 2    50   Input ~ 0
 CAN_TX_2
-Text HLabel 6900 5050 2    50   Output ~ 0
+Text HLabel 5400 3550 2    50   Output ~ 0
 CAN_RX_2
 $Comp
@@
 	0    1    1    0
 $EndComp
-Text Notes 6500 4550 0    59   ~ 0
+Text Notes 5000 3050 0    59   ~ 0
 USE CAN1/CAN2 and CAN3
 Wire Wire Line
@@
 Wire Notes Line
 	9000 850  9000 3250
-Text Notes 6500 5650 0    59   ~ 0
+Text Notes 5000 4150 0    59   ~ 0
 USE SPI1,4,5,6 for 54 Mbps
 Text Label 5200 2750 2    59   ~ 0
 SWCLK
-Text Label 5200 2850 2    59   ~ 0
+Text Label 5525 2825 2    59   ~ 0
 SWDIO
 Wire Wire Line
 	4550 2750 5200 2750
 Wire Wire Line
-	4550 2850 5200 2850
+	4875 2825 5525 2825
 Text Notes 11950 6800 0    59   ~ 0
 Debug leds\n
@@
 Wire Notes Line
 	13400 9450 13400 6850
-Text HLabel 6900 6300 2    59   Output ~ 0
+Text HLabel 5400 4800 2    59   Output ~ 0
 HGM
-Text HLabel 6900 6400 2    59   Output ~ 0
+Text HLabel 5400 4900 2    59   Output ~ 0
 LNA_EN
-Text HLabel 6900 6500 2    59   Output ~ 0
+Text HLabel 5400 5000 2    59   Output ~ 0
 PA_EN
-Text HLabel 6900 6950 2    59   BiDi ~ 0
+Text HLabel 5400 5450 2    59   BiDi ~ 0
 RF_GPIO0
-Text HLabel 6900 6850 2    59   BiDi ~ 0
+Text HLabel 5400 5350 2    59   BiDi ~ 0
 RF_GPIO2
-Text HLabel 6900 6750 2    59   BiDi ~ 0
+Text HLabel 5400 5250 2    59   BiDi ~ 0
 RF_GPIO3
 $EndSCHEMATC

Commit message: Added MCU config pins
Parts:
- added C?: C, symbol Device:C
Connections:
- net +3V3: now also U5.100 (VCAPDSI), U5.38 (VREF+), C?.1
- net BOOT0: now also U5.166 (BOOT0)
- net BYPASS_REG: now also U5.48 (BYPASS_REG)
- net CAN_RX_1: now also U5.168 (PB9)
- net CAN_RX_2: now also U5.161 (PB3)
- net CAN_TX_1: now also U5.167 (PB8)
- net CAN_TX_2: now also U5.162 (PB4)
- net CAP_1: now also U5.81 (VCAP_1)
- net CAP_2: now also U5.129 (VCAP_2)
- net GND: now also C?.2
- net HGM: now also U5.32 (PC0)
- net LED_1: now also U5.121 (PC8)
- net LED_2: now also U5.122 (PC9)
- net LED_3: now also U5.139 (PC10)
- net LNA_EN: now also U5.33 (PC1)
- net MISO: now also U5.52 (PA6)
- net MOSI: now also U5.53 (PA7)
- net NRST: now also U5.31 (NRST)
- net PA_EN: now also U5.34 (PC2)
- net PDR_ON: now also U5.171 (PDR_ON)
- net RF_GPIO0: now also U5.55 (PC5)
- net RF_GPIO2: now also U5.54 (PC4)
- net RF_GPIO3: now also U5.35 (PC3)
- net SLCK: now also U5.51 (PA5)
- net SWDIO: now also U5.137 (PA14)
- net ~CS: now also U5.50 (PA4)
Other:
- note added: "CAN1"
- note added: "CAN3\n\n"
- note added: "SPI1"
- note removed: "USE CAN1/CAN2 and CAN3"
- note removed: "USE SPI1,4,5,6 for 54 Mbps"
Changed lines of the file:
@@
 Comment4 ""
 $EndDescr
-Text HLabel 5400 4250 2    59   Output ~ 0
+Text HLabel 4950 1950 2    59   Output ~ 0
 SLCK
-Text HLabel 5400 4350 2    59   Output ~ 0
+Text HLabel 4950 2150 2    59   Output ~ 0
 MOSI
-Text HLabel 5400 4450 2    59   Input ~ 0
+Text HLabel 4950 2050 2    59   Input ~ 0
 MISO
-Text HLabel 5400 4550 2    59   Output ~ 0
+Text HLabel 4950 1850 2    59   Output ~ 0
 ~CS
 $Comp
@@
 	1    0    0    -1
 $EndComp
-Text HLabel 5400 3150 2    50   Input ~ 0
+Text HLabel 4950 3950 2    50   Input ~ 0
 CAN_TX_1
-Text HLabel 5400 3250 2    50   Output ~ 0
+Text HLabel 4950 4050 2    50   Output ~ 0
 CAN_RX_1
-Text HLabel 5400 3450 2    50   Input ~ 0
+Text HLabel 4950 3550 2    50   Input ~ 0
 CAN_TX_2
-Text HLabel 5400 3550 2    50   Output ~ 0
+Text HLabel 4950 3450 2    50   Output ~ 0
 CAN_RX_2
 $Comp
@@
 	0    1    1    0
 $EndComp
-Text Notes 5000 3050 0    59   ~ 0
-USE CAN1/CAN2 and CAN3
 Wire Wire Line
 	2550 10050 2650 10050
@@
 Wire Notes Line
 	9000 850  9000 3250
-Text Notes 5000 4150 0    59   ~ 0
-USE SPI1,4,5,6 for 54 Mbps
-Text Label 5200 2750 2    59   ~ 0
+Text Label 5700 2750 2    59   ~ 0
 SWCLK
-Text Label 5525 2825 2    59   ~ 0
-SWDIO
-Wire Wire Line
-	4550 2750 5200 2750
-Wire Wire Line
-	4875 2825 5525 2825
 Text Notes 11950 6800 0    59   ~ 0
 Debug leds\n
@@
 Wire Notes Line
 	13400 9450 13400 6850
-Text HLabel 5400 4800 2    59   Output ~ 0
+Text HLabel 4950 4850 2    59   Output ~ 0
 HGM
-Text HLabel 5400 4900 2    59   Output ~ 0
+Text HLabel 4950 4950 2    59   Output ~ 0
 LNA_EN
-Text HLabel 5400 5000 2    59   Output ~ 0
+Text HLabel 4950 5050 2    59   Output ~ 0
 PA_EN
-Text HLabel 5400 5450 2    59   BiDi ~ 0
+Text HLabel 4950 5350 2    59   BiDi ~ 0
 RF_GPIO0
-Text HLabel 5400 5350 2    59   BiDi ~ 0
+Text HLabel 4950 5250 2    59   BiDi ~ 0
 RF_GPIO2
-Text HLabel 5400 5250 2    59   BiDi ~ 0
+Text HLabel 4950 5150 2    59   BiDi ~ 0
 RF_GPIO3
+Text Label 5700 2850 2    59   ~ 0
+SWDIO
+Wire Wire Line
+	4950 1850 4550 1850
+Wire Wire Line
+	4550 1950 4950 1950
+Wire Wire Line
+	4550 2050 4950 2050
+Wire Wire Line
+	4550 2150 4950 2150
+Wire Wire Line
+	4550 3950 4950 3950
+Wire Wire Line
+	4550 4050 4950 4050
+Wire Wire Line
+	4550 2750 5700 2750
+Wire Wire Line
+	4550 2850 5700 2850
+Wire Wire Line
+	4550 3450 4950 3450
+Wire Wire Line
+	4550 3550 4950 3550
+Text Notes 5450 4000 0    59   ~ 0
+CAN1
+Text Notes 5450 3600 0    59   ~ 0
+CAN3\n\n
+Text Notes 5400 1850 0    59   ~ 0
+SPI1
+Wire Wire Line
+	4550 4850 4950 4850
+Wire Wire Line
+	4550 4950 4950 4950
+Wire Wire Line
+	4550 5050 4950 5050
+Wire Wire Line
+	4550 5150 4950 5150
+Wire Wire Line
+	4550 5250 4950 5250
+Wire Wire Line
+	4550 5350 4950 5350
+Text Label 5700 5650 2    59   ~ 0
+LED_1
+Text Label 5700 5750 2    59   ~ 0
+LED_2
+Text Label 5700 5850 2    59   ~ 0
+LED_3
+Wire Wire Line
+	4550 5650 5700 5650
+Wire Wire Line
+	4550 5750 5700 5750
+Wire Wire Line
+	4550 5850 5700 5850
+Text Label 1250 1450 2    59   ~ 0
+NRST
+Text Label 1250 1550 2    59   ~ 0
+BYPASS_REG
+Text Label 1250 1850 2    59   ~ 0
+BOOT0
+Text Label 1250 1650 2    59   ~ 0
+PDR_ON
+Text Label 1250 2050 2    59   ~ 0
+CAP_DSI
+Text Label 1250 2150 2    59   ~ 0
+CAP_1
+Text Label 1250 2250 2    59   ~ 0
+CAP_2
+Wire Wire Line
+	700  2350 700  2175
+$Comp
+L power:+3.3V #PWR?
+U 1 1 60304CA3
+P 700 2175
+F 0 "#PWR?" H 700 2025 50  0001 C CNN
+F 1 "+3.3V" H 715 2348 50  0000 C CNN
+F 2 "" H 700 2175 50  0001 C CNN
+F 3 "" H 700 2175 50  0001 C CNN
+	1    700  2175
+	1    0    0    -1
+$EndComp
+Wire Wire Line
+	700  2350 1450 2350
+Wire Wire Line
+	1250 1450 1450 1450
+Wire Wire Line
+	1250 1550 1450 1550
+Wire Wire Line
+	1250 1650 1450 1650
+Wire Wire Line
+	1250 1850 1450 1850
+Wire Wire Line
+	1450 2050 1250 2050
+Wire Wire Line
+	1450 2150 1250 2150
+Wire Wire Line
+	1450 2250 1250 2250
+$Comp
+L Device:C C?
+U 1 1 6034349C
+P 4825 1300
+F 0 "C?" H 4940 1346 50  0000 L CNN
+F 1 "C" H 4940 1255 50  0000 L CNN
+F 2 "" H 4863 1150 50  0001 C CNN
+F 3 "~" H 4825 1300 50  0001 C CNN
+	1    4825 1300
+	1    0    0    -1
+$EndComp
+$Comp
+L power:GND #PWR?
+U 1 1 603444EA
+P 4825 1450
+F 0 "#PWR?" H 4825 1200 50  0001 C CNN
+F 1 "GND" H 4830 1277 50  0000 C CNN
+F 2 "" H 4825 1450 50  0001 C CNN
+F 3 "" H 4825 1450 50  0001 C CNN
+	1    4825 1450
+	1    0    0    -1
+$EndComp
+Wire Wire Line
+	4050 1150 4825 1150
+Text Label 4825 1150 2    59   ~ 0
+CAP_DSI
 $EndSCHEMATC

Commit message: Changes to PA layout
Parts:
- added C?: 1u, Capacitor_SMD:C_0603_1608Metric, symbol Device:C
- added C?: 100n, Capacitor_SMD:C_0603_1608Metric, symbol Device:C
- C18: renamed from C?; footprint (none) -> Capacitor_SMD:C_0603_1608Metric
- C33, C34, C35, C36, C37, C38, C39, C40, C41, C42, C43, C44, C45, C47, C49, C50, C51, C52, C53, C54, C56: footprint (none) -> Capacitor_SMD:C_0603_1608Metric
- C46: value 100n -> 2.2u; footprint (none) -> Capacitor_SMD:C_0603_1608Metric
- C48: value C -> 2.2u; footprint (none) -> Capacitor_SMD:C_0603_1608Metric
- R1, R2, R8: value R -> 1k; footprint (none) -> Resistor_SMD:R_0603_1608Metric
- R10, R11, R12, R9: footprint (none) -> Resistor_SMD:R_0603_1608Metric
Connections:
- net +3V3: now also C?.1, C?.1
- net GND: now also C?.2, C?.2
- net ~CS_1: now reaches U5.47 (PA3)
- net ~CS renamed ~CS_2
Other:
- note added: "VREF\n"
